File: bandpass_filter.kicad_pcb (KiCad board)
At the start: 2 copper layers, 94 x 25.4 mm, 22 parts, among them J1 PCB.SMAFRA.HT, J3 PCB.SMAFRA.HT

Commit message: Add spice model.
Parts:
- R1, R2: value 50 Ohms -> r=50
Connections:
- net Net-(J1-Pad1) renamed V_out
- net Net-(J3-Pad1) renamed V_in
Changed lines of the file:
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@@
   (net 9 "Net-(C9-Pad1)")
   (net 10 "GND")
-  (net 11 "Net-(J1-Pad1)")
-  (net 12 "Net-(J3-Pad1)")
+  (net 11 "V_out")
+  (net 12 "V_in")
   (footprint "Inductor_SMD:L_1206_3216Metric" (layer "F.Cu")
     (at 73.985565 61.565476 -90)
@@
     (property "Sheetfile" "bandpass_filter.kicad_sch")
     (property "Sheetname" "")
+    (property "Sim.Device" "R")
+    (property "Sim.Params" "r=50")
+    (property "Sim.Pins" "1=+ 2=-")
+    (property "Sim.Type" "=")
     (property "ki_description" "Resistor, US symbol")
     (property "ki_keywords" "R res resistor")
@@
         (effects (font (size 1 1) (thickness 0.15)))
     )
-    (fp_text value "50 Ohms" (at 0 1.82) (layer "F.Fab") hide
+    (fp_text value "r=50" (at 0 1.82) (layer "F.Fab") hide
         (effects (font (size 1 1) (thickness 0.15)))
     )
@@
       (stroke (width 0.1) (type solid)) (layer "F.Fab"))
     (pad "1" smd roundrect (at -1.4625 0) (size 1.125 1.75) (layers "F.Cu" "F.Paste" "F.Mask") (roundrect_rratio 0.2222222222)
-      (net 12 "Net-(J3-Pad1)") (pintype "passive"))
+      (net 12 "V_in") (pintype "passive"))
     (pad "2" smd roundrect (at 1.4625 0) (size 1.125 1.75) (layers "F.Cu" "F.Paste" "F.Mask") (roundrect_rratio 0.2222222222)
       (net 1 "Net-(C1-Pad1)") (pintype "passive"))
@@
     (property "Sheetfile" "bandpass_filter.kicad_sch")
     (property "Sheetname" "")
+    (property "Sim.Enable" "0")
     (property "ki_description" "RF Connectors / Coaxial Connectors SMA RA PCB Mount, Jack, Gold, 50 , Through Hole Pin")
     (attr through_hole)
@@
       (stroke (width 0.2) (type solid)) (layer "F.Fab"))
     (pad "1" thru_hole circle (at 0 0) (size 2.4 2.4) (drill 1.6) (layers "*.Cu" "*.Mask")
-      (net 12 "Net-(J3-Pad1)") (pinfunction "1") (pintype "passive"))
+      (net 12 "V_in") (pinfunction "1") (pintype "passive"))
     (pad "2" thru_hole circle (at -2.575 -2.575) (size 2.85 2.85) (drill 1.9) (layers "*.Cu" "*.Mask")
       (net 10 "GND") (pinfunction "2") (pintype "passive"))
@@
     (property "Sheetfile" "bandpass_filter.kicad_sch")
     (property "Sheetname" "")
+    (property "Sim.Enable" "0")
     (property "ki_description" "RF Connectors / Coaxial Connectors SMA RA PCB Mount, Jack, Gold, 50 , Through Hole Pin")
     (attr through_hole)
@@
       (stroke (width 0.2) (type solid)) (layer "F.Fab"))
     (pad "1" thru_hole circle (at 0 0) (size 2.4 2.4) (drill 1.6) (layers "*.Cu" "*.Mask")
-      (net 11 "Net-(J1-Pad1)") (pinfunction "1") (pintype "passive"))
+      (net 11 "V_out") (pinfunction "1") (pintype "passive"))
     (pad "2" thru_hole circle (at -2.575 -2.575) (size 2.85 2.85) (drill 1.9) (layers "*.Cu" "*.Mask")
       (net 10 "GND") (pinfunction "2") (pintype "passive"))
@@
     (property "Sheetfile" "bandpass_filter.kicad_sch")
     (property "Sheetname" "")
+    (property "Sim.Device" "R")
+    (property "Sim.Params" "r=50")
+    (property "Sim.Pins" "1=+ 2=-")
+    (property "Sim.Type" "=")
     (property "ki_description" "Resistor, US symbol")
     (property "ki_keywords" "R res resistor")
@@
         (effects (font (size 1 1) (thickness 0.15)))
     )
-    (fp_text value "50 Ohms" (at 0 1.82) (layer "F.Fab") hide
+    (fp_text value "r=50" (at 0 1.82) (layer "F.Fab") hide
         (effects (font (size 1 1) (thickness 0.15)))
     )
@@
       (net 9 "Net-(C9-Pad1)") (pintype "passive"))
     (pad "2" smd roundrect (at 1.4625 0) (size 1.125 1.75) (layers "F.Cu" "F.Paste" "F.Mask") (roundrect_rratio 0.2222222222)
-      (net 11 "Net-(J1-Pad1)") (pintype "passive"))
+      (net 11 "V_out") (pintype "passive"))
     (model "${KICAD6_3DMODEL_DIR}/Resistor_SMD.3dshapes/R_1206_3216Metric.wrl"
       (offset (xyz 0 0 0))
